File: STARDANCE-HACKPAD.kicad_pcb (KiCad board)
At the start: 2 copper layers, 3.6 x 3.2 mm, 8 parts, among them J1 Conn_01x04_Socket, SW2 SW_Push, SW3 SW_Push, SW4 SW_Push, U1 MOUDLE-SEEEDUINO-XIAO

Commit message: Journaling and KiCad for 7/12/2026
Parts:
- moved SW3 0.50 mm to (138.5, 111.4)
Routing:
- net +5V: track 69.4 -> 198.4 mm
- net /LEDDATA: track 68.4 -> 117.7 mm
- net /B3: track 26.2 -> 62.5 mm
- net GND: track 259.6 -> 230.8 mm
- net Net-(D2-DOUT): track 0.00 -> 22.7 mm
- net /SDA: track 99.8 -> 79.8 mm
- net /SCL: track 86.7 -> 95.6 mm
- net Net-(D1-DOUT): track 87.3 -> 94.9 mm
- net +3.3V: track 77.0 -> 74.4 mm

Commit message: 7/13/2026
Parts:
- moved D1 7.69 mm to (104.5, 125.8)
- moved D2 7.69 mm to (156.0, 125.8)
- moved D3 7.69 mm to (128.5, 125.8)
- moved J1 7.69 mm to (94.5, 70.5)
- moved SW2 7.69 mm to (106.0, 108.2)
- moved SW3 7.69 mm to (131.5, 108.2)
- moved SW4 7.69 mm to (158.0, 108.2)
- moved U1 7.69 mm to (168.2, 92.8)
Routing:
- net GND: track 230.8 -> 216.9 mm
- added copper zone on B.Cu, net GND
Other:
- board size 3.6 x 3.2 mm -> 101.5 x 80.5 mm

Commit message: Journaled 7/16/26 finished PCB
Routing:
- removed copper zone on B.Cu, net GND
Changed lines of the file:
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@@
 		(capping no)
 		(filling no)
-		(zone_defaults)
 		(pcbplotparams
 			(layerselection 0x00000000_00000000_55555555_575555ff)
@@
 		(net "/B2")
 	)
-	(zone
-		(net "GND")
-		(layer "B.Cu")
-		(hatch edge 0.5)
-		(connect_pads
-			(clearance 0.5)
-		)
-		(min_thickness 0.25)
-		(fill yes
-			(thermal_gap 0.5)
-			(thermal_bridge_width 0.5)
-			(island_removal_mode 0)
-		)
-		(polygon
-			(pts
-				(xy 83.5 59.5) (xy 83.5 140) (xy 185 140) (xy 185 59.5)
-			)
-		)
-	)
 	(embedded_fonts no)
